Commit message: zmiana inercji zeby dron byl bardziej snapy, do sprawdzenia

File: simulation/drone_models/cf2x/cf2x.urdf (robot description, URDF)
Before this commit: robot cf2, 7 links, 6 joints
Links:
- link base_link: mass 0.07 -> 0.025

Commit message: Added testing env with radio

File: simulation/drone_models/cf2x/cf2x.urdf (robot description, URDF)
Before this commit: robot cf2, 7 links, 6 joints
Links:
- link base_link: mass 0.025 -> 0.1
